Commit message: feat: move robot node

File: roboturo/urdf/robo.urdf (robot description, URDF)
Before this commit: robot robot_uro, 5 links, 4 joints
Links:
- removed link back-left-wheel
- removed link back-right-wheel
- removed link base
- removed link front-left-wheel
- removed link front-right-wheel
- added link base_link; visual box size=0.5 0.5 0.1
- added link left_wheel, mass 0.5; collision cylinder length=0.05 radius=0.1; visual cylinder length=0.05 radius=0.1
- added link right_wheel, mass 0.5; collision cylinder length=0.05 radius=0.1; visual cylinder length=0.05 radius=0.1
Joints:
- removed joint back-left-joint
- removed joint back-right-joint
- removed joint front-left-joint
- removed joint front-right-joint
- added joint left_wheel_joint: type continuous, parent base_link, child left_wheel, origin xyz=0 0.3 0 rpy=0 0 0
- added joint right_wheel_joint: type continuous, parent base_link, child right_wheel, origin xyz=0 -0.3 0 rpy=0 0 0
